Commit message: Fixed gazebo sim, added slam mapping

File: description/gazebo_control.xacro (robot description, xacro)
@@ -6,6 +6,6 @@
             <left_joint>left_wheel_joint</left_joint>
             <right_joint>right_wheel_joint</right_joint>
-            <wheel_separation>0.140</wheel_separation>
-            <wheel_radius>0.033</wheel_radius>
+            <wheel_separation>0.155</wheel_separation>
+            <wheel_radius>0.0325</wheel_radius>
             <!--LIMITS-->
             <!-- <max_wheel_torque>200</max_wheel_torque> -->

File: description/robot.urdf.xacro (robot description, xacro)
@@ -2,5 +2,5 @@
 <robot xmlns:xacro="http://www.ros.org/wiki/xacro"  name="robot">
     <xacro:arg name="use_ros2_control" default="true"/>
-    <xacro:arg name="sim_mode" default="false"/>
+    <xacro:arg name="sim_mode" default="true"/>
     <xacro:include filename="robot_core.xacro" />
     <xacro:if value="$(arg use_ros2_control)">

File: description/robot_core.xacro (robot description, xacro)
@@ -20,4 +20,12 @@
     <!--BASE LINK (standard to do in ROS)-->
     <link name="base_link">
+    </link>
+    <!--BASE FOOTPRINT LINK-->
+    <joint name="base_footprint_joint" type="fixed">
+        <parent link="base_link"/>
+        <child link="base_footprint"/>
+        <origin xyz="0 0 0" rpy="0 0 0"/>
+    </joint>
+    <link name="base_footprint">
     </link>
     <!--CHASSIS LINK-->
